File: TGC-Core-ULTRA32-v1.kicad_sch (KiCad schematic)
At the start: 32 parts, among them J1 Conn_01x19, J2 Conn_01x19, P1 USB_C_Plug_USB2.0, Q1 SS8050-G, Q2 SS8050-G, SW1 SW_Push, SW2 SW_Push, U1 CP2102N-Axx-xQFN28, U2 AMS1117-3.3

Commit message: Add files via upload
Other:
- note added: "USB to Serial"
Changed lines of the file:
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@@
 	(generator_version "10.0")
 	(paper "A4")
+	(text "USB to Serial"
+		(exclude_from_sim no)
+		(at 151.892 97.79 0)
+		(effects
+			(font
+				(size 1.27 1.27)
+				(thickness 0.254)
+				(bold yes)
+			)
+		)
+	)
 	(junction
 		(at 90.17 99.06)
